File: Pico_VGA_Board/Pico_VGA_Board/Pico_VGA_Board.kicad_pcb (KiCad board)
At the start: 2 copper layers, 80 x 60 mm, 56 parts, among them IC1 NC7WZ17P6X, J1 DE15_Plug_HighDensity, J2 Micro_SD_Card_Det1, J3 AudioJack3, SW1 SW_MEC_5E, U1 Pico

Commit message: Beeren an da Rückseitn pflanzt
Parts:
- added G***: LOGO, Symbol:VGA, B.Cu at (155.0, 92.0)
- added G***: LOGO, Symbol:RasPi, B.Cu at (155.0, 75.8)
Other:
- board text added: "x"

Commit message: Update Pico_VGA_Board.kicad_pcb
Parts:
- moved TP1 4.01 mm to (133.8, 77.5)
- moved TP2 1.03 mm to (133.8, 85.0)
- moved R17 1.00 mm to (137.5, 107.5)
- moved G*** 0.50 mm to (130.5, 64.0)
- moved TP11 0.25 mm to (171.2, 82.5)
- moved TP3 0.25 mm to (133.8, 92.5)
Routing:
- net /VGA_B: track 22.0 -> 24.8 mm
- net /VGA_G: track 22.6 -> 20.6 mm
- net /SD_CLK: track 71.3 -> 69.8 mm
- net GND: vias 122 -> 173
Other:
- board text added: "B"
- board text added: "G"
- board text added: "H"
- board text added: "R"
- board text added: "V"

Commit message: Stitching DK
Routing:
- net GND: track 12.8 -> 11.1 mm, vias 173 -> 176
- net /VGA_B: track 24.8 -> 25.6 mm
- net /VGA_G: track 20.6 -> 19.9 mm

Commit message: Silkscreen Pins
Routing:
- net /SD_DAT0: track 33.3 -> 34.4 mm
- net /SD_DAT2: track 32.4 -> 31.8 mm
Other:
- board text added: "CMD"
- board text added: "D0"
- board text added: "D1"
- board text added: "D2"
- board text added: "D3"

Commit message: upd Silkscreen
Parts:
- removed the G*** at (130.5, 64.0)
- added G***: LOGO, Symbol:Speaker_2.5x2.5, F.Cu at (169.8, 72.4)
- added G***: LOGO, Symbol:VGA_RGB, F.Cu at (130.0, 64.0)
- added G***: LOGO, Symbol:Speaker_2.5x2.5, F.Cu at (169.8, 77.4)
- moved TP11 0.34 mm to (171.4, 82.2)
Other:
- board text added: "+"
- board text added: "CLK"
- board text added: "L"

Commit message: Sound Control 2 Versions
Parts:
- R24: value 220 -> 220R
- R26: value 100 -> 100R
Changed lines of the file:
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@@
         (effects (font (size 1 1) (thickness 0.15)))
     )
-    (fp_text value "Dim" (at 0 1.43) (layer "F.Fab")
+    (fp_text value "Dim" (at 0 -1.5) (layer "F.Fab")
         (effects (font (size 1 1) (thickness 0.15)))
     )
@@
         (effects (font (size 1 1) (thickness 0.15)))
     )
-    (fp_text value "SW_MEC_5E" (at 3.2 6.5 90) (layer "F.Fab")
+    (fp_text value "SW_MEC_5E" (at 0.55 -2.4 270) (layer "F.Fab")
         (effects (font (size 1 1) (thickness 0.15)))
     )
@@
         (effects (font (size 1 1) (thickness 0.15)))
     )
-    (fp_text value "TestPoint" (at 0 2.05) (layer "F.Fab")
+    (fp_text value "TestPoint" (at 0 2.3) (layer "F.Fab")
         (effects (font (size 1 1) (thickness 0.15)))
     )
@@
         (effects (font (size 1 1) (thickness 0.15)))
     )
-    (fp_text value "220" (at 0 1.43) (layer "F.Fab")
+    (fp_text value "220R" (at 3.4 0) (layer "F.Fab")
         (effects (font (size 1 1) (thickness 0.15)))
     )
@@
         (effects (font (size 1 1) (thickness 0.15)))
     )
-    (fp_text value "100n" (at 0 1.43) (layer "F.Fab")
+    (fp_text value "100n" (at -3.3 0.2) (layer "F.Fab")
         (effects (font (size 1 1) (thickness 0.15)))
     )
@@
         (effects (font (size 1 1) (thickness 0.15)))
     )
-    (fp_text value "AudioJack3" (at 0 13 90) (layer "F.Fab")
+    (fp_text value "AudioJack3" (at 3.9 4.3 -180) (layer "F.Fab")
         (effects (font (size 1 1) (thickness 0.15)))
     )
@@
         (effects (font (size 1 1) (thickness 0.15)))
     )
-    (fp_text value "47u" (at 0 1.43) (layer "F.Fab")
+    (fp_text value "47u" (at -3 0) (layer "F.Fab")
         (effects (font (size 1 1) (thickness 0.15)))
     )
@@
         (effects (font (size 1 1) (thickness 0.15)))
     )
-    (fp_text value "100" (at 0 1.43) (layer "F.Fab")
+    (fp_text value "100R" (at 3.5 -0.1) (layer "F.Fab")
         (effects (font (size 1 1) (thickness 0.15)))
     )
@@
         (effects (font (size 1 1) (thickness 0.15)))
     )
-    (fp_text value "LED" (at 0 1.82) (layer "F.Fab")
+    (fp_text value "LED" (at -3.6 0) (layer "F.Fab")
         (effects (font (size 1 1) (thickness 0.15)))
     )
@@
         (effects (font (size 1 1) (thickness 0.15)))
     )
-    (fp_text value "Dim" (at 0 1.43) (layer "F.Fab")
+    (fp_text value "Dim" (at 0.1 -1.5) (layer "F.Fab")
         (effects (font (size 1 1) (thickness 0.15)))
     )
@@
         (effects (font (size 1 1) (thickness 0.15)))
     )
-    (fp_text value "1.8k" (at 0 1.43) (layer "F.Fab")
+    (fp_text value "1.8k" (at -3.2 0.1) (layer "F.Fab")
         (effects (font (size 1 1) (thickness 0.15)))
     )
@@
   (segment (start 183.95 78.325) (end 184 78.275) (width 0.3) (layer "F.Cu") (net 3))
   (segment (start 178 78.325) (end 183.95 78.325) (width 0.3) (layer "F.Cu") (net 3))
-  (segment (start 190.1 73.9) (end 190.1 73.7) (width 0.3) (layer "F.Cu") (net 4))
+  (segment (start 187.325 76.675) (end 190.1 73.9) (width 0.3) (layer "F.Cu") (net 4))
   (segment (start 184 76.725) (end 185.95 76.725) (width 0.3) (layer "F.Cu") (net 4))
   (segment (start 186 76.675) (end 187.325 76.675) (width 0.3) (layer "F.Cu") (net 4))
-  (segment (start 187.325 76.675) (end 190.1 73.9) (width 0.3) (layer "F.Cu") (net 4))
+  (segment (start 190.1 73.9) (end 190.1 73.7) (width 0.3) (layer "F.Cu") (net 4))
   (segment (start 185.95 76.725) (end 186 76.675) (width 0.3) (layer "F.Cu") (net 4))
   (segment (start 174.225 69) (end 174.225 74.95) (width 0.3) (layer "F.Cu") (net 5))
