File: Pico_VGA_Board/Pico_VGA_Board/Pico_VGA_Board.kicad_sch (KiCad schematic)
At the start: 51 parts, among them IC1 NC7WZ17P6X, J1 DE15_Plug_HighDensity, J2 Micro_SD_Card_Det1, J3 AudioJack3, SW1 SW_MEC_5E, U1 Pico

Commit message: UPD Board
Parts:
- added H1, H2, H3, H4: MountingHole_Pad, MountingHole:MountingHole_3.2mm_M3_Pad_Via, symbol Mechanical:MountingHole_Pad
- IC1: footprint SOP65P210X110-6N -> SamacSys_Parts:SOP65P210X110-6N
- J2: footprint Samacsys:5033981892 -> SamacSys_Parts:503398-1892
- J3: footprint Connector_Audio:Jack_3.5mm_CUI_SJ-3523-SMT_Horizontal -> Connector_Audio:Jack_3.5mm_CUI_SJ-3524-SMT_Horizontal
- U1: footprint Pico_W:RPi_Pico_SMD_TH -> Module:RPi_Pico_SMD_TH
Connections:
- net +3V3: now also R23.2; no longer D2.2 (A)
- net GND: now also D2.1 (K), D3.1 (K), H1.1, H2.1, H3.1, H4.1; no longer R23.2, R30.2
- net SD_ERR_LED: now also R30.1; no longer D3.2 (A)
- net at R23.1: now also D2.2 (A); no longer D2.1 (K)
- new net: D3.2 (A), R30.2
- no-connect marks 0 -> 7
Other:
- moved on the sheet: D2, D3, J3, R23, R30

Commit message: 1-Heiten
Parts:
- J3: value AudioJack3 -> PWM-Audio
- R1, R11, R6: value 499 -> 499R
- R10, R15, R5: value 8.06k -> 8k06
- R14, R4, R9: value 4.02k -> 4k02
- R16, R17: value 47 -> 47R
- R24, R25: value 220 -> 220R
- R26, R27: value 100 -> 100R
- R28, R29: value 1.8k -> 1k8
Other:
- moved on the sheet: C2, C3, C4, C5, C6, D1, J3, R18, R19, R20, R21, R24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

Commit message: update
Parts:
- J3: LCSC Part # C4991872 -> C4991872
Changed lines of the file:
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@@
       (effects (font (size 1.27 1.27)) hide)
     )
-    (property "LCSC Part #" " C4991872 " (at 257.81 140.97 0)
+    (property "LCSC Part #" "C4991872 " (at 257.81 140.97 0)
       (effects (font (size 1.27 1.27)) hide)
     )
