File: SoundControl/PCB/SoundControl.kicad_pcb (KiCad board)
At the start: 2 copper layers, 101.6 x 101.6 mm, 38 parts, among them SW1 SW_Push, SW2 SW_Push, SW3 SW_Push, SW4 SW_Push, SW5 SW_Push, U1 CD4051BCN, U2 Pico

Commit message: firmware and pinout
Connections:
- U2 pad 36: unconnected-(U2-3V3-Pad36) -> +3V3
Other:
- board size 101.6 x 101.6 mm -> 101.6 x 99.1 mm
Changed lines of the file:
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@@
   (net 47 "unconnected-(U2-GPIO28_ADC2-Pad34)")
   (net 48 "unconnected-(U2-ADC_VREF-Pad35)")
-  (net 49 "unconnected-(U2-3V3-Pad36)")
-  (net 50 "unconnected-(U2-3V3_EN-Pad37)")
-  (net 51 "unconnected-(U2-VSYS-Pad39)")
+  (net 49 "unconnected-(U2-3V3_EN-Pad37)")
+  (net 50 "unconnected-(U2-VSYS-Pad39)")
   (footprint "Resistor_THT:R_Axial_DIN0207_L6.3mm_D2.5mm_P10.16mm_Horizontal" (layer "F.Cu")
     (at 134.62 144.78 90)
@@
       (net 48 "unconnected-(U2-ADC_VREF-Pad35)") (pinfunction "ADC_VREF") (pintype "power_in"))
     (pad "36" thru_hole oval (at 8.89 -13.97) (size 1.7 1.7) (drill 1.02) (layers "*.Cu" "*.Mask")
-      (net 49 "unconnected-(U2-3V3-Pad36)") (pinfunction "3V3") (pintype "power_in"))
+      (net 13 "+3V3") (pinfunction "3V3") (pintype "power_in"))
     (pad "37" thru_hole oval (at 8.89 -16.51) (size 1.7 1.7) (drill 1.02) (layers "*.Cu" "*.Mask")
-      (net 50 "unconnected-(U2-3V3_EN-Pad37)") (pinfunction "3V3_EN") (pintype "input"))
+      (net 49 "unconnected-(U2-3V3_EN-Pad37)") (pinfunction "3V3_EN") (pintype "input"))
     (pad "38" thru_hole rect (at 8.89 -19.05) (size 1.7 1.7) (drill 1.02) (layers "*.Cu" "*.Mask")
       (net 1 "GND") (pinfunction "GND") (pintype "bidirectional"))
     (pad "39" thru_hole oval (at 8.89 -21.59) (size 1.7 1.7) (drill 1.02) (layers "*.Cu" "*.Mask")
-      (net 51 "unconnected-(U2-VSYS-Pad39)") (pinfunction "VSYS") (pintype "power_in"))
+      (net 50 "unconnected-(U2-VSYS-Pad39)") (pinfunction "VSYS") (pintype "power_in"))
     (pad "40" thru_hole oval (at 8.89 -24.13) (size 1.7 1.7) (drill 1.02) (layers "*.Cu" "*.Mask")
       (net 3 "+5V") (pinfunction "VBUS") (pintype "power_in"))
@@
     )
   )
-  (gr_rect (start 101.6 52.07) (end 203.2 153.67)
+  (gr_rect (start 101.6 52.07) (end 203.2 151.13)
     (stroke (width 0.1) (type default)) (fill none) (layer "Edge.Cuts"))
   (segment (start 154.94 142.24) (end 170.18 142.24) (width 0.5) (layer "B.Cu") (net 1))
