File: SoundControl/PCB/SoundControl.kicad_sch (KiCad schematic)
At the start: 38 parts, among them SW1 SW_Push, SW2 SW_Push, SW3 SW_Push, SW4 SW_Push, SW5 SW_Push, U1 CD4051BCN, U2 Pico

Commit message: firmware and pinout
Connections:
- net +3V3: now also U2.36 (3V3)
- no-connect marks 0 -> 1
Changed lines of the file:
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@@
   (junction (at 190.5 49.53) (diameter 0) (color 0 0 0 0)
   )
+  (no_connect (at 285.75 35.56))
   (wire (pts (xy 207.01 64.77) (xy 210.82 64.77))
     (stroke (width 0) (type default))
@@
     (stroke (width 0) (type default))
   )
+  (wire (pts (xy 270.51 33.02) (xy 270.51 41.91))
+    (stroke (width 0) (type default))
+  )
   (wire (pts (xy 207.01 52.07) (xy 210.82 52.07))
     (stroke (width 0) (type default))
@@
   )
   (wire (pts (xy 118.11 110.49) (xy 121.92 110.49))
+    (stroke (width 0) (type default))
+  )
+  (wire (pts (xy 246.38 41.91) (xy 270.51 41.91))
     (stroke (width 0) (type default))
   )
@@
   )
   (symbol (lib_id "Device:R") (at 71.12 119.38 0) (unit 1)
-    (in_bom yes) (on_board yes) (dnp no) (fields_autoplaced)
+    (in_bom yes) (on_board yes) (dnp no)
     (property "Reference" "R3" (at 73.66 118.745 0)
       (effects (font (size 1.27 1.27)) (justify left))
@@
         )
       )
+    )
+  )
+  (symbol (lib_id "power:+3V3") (at 270.51 33.02 0) (unit 1)
+    (in_bom yes) (on_board yes) (dnp no) (fields_autoplaced)
+    (property "Reference" "#PWR033" (at 270.51 36.83 0)
+      (effects (font (size 1.27 1.27)) hide)
+    )
+    (property "Value" "+3V3" (at 270.51 29.21 0)
+      (effects (font (size 1.27 1.27)))
+    )
+    (property "Footprint" "" (at 270.51 33.02 0)
+      (effects (font (size 1.27 1.27)) hide)
+    )
+    (property "Datasheet" "" (at 270.51 33.02 0)
+      (effects (font (size 1.27 1.27)) hide)
+    )
+    (pin "1")
+    (instances
+      (project "SoundControl"
+        (path "/06c37cb1-c02e-4807-841e-a1362f60cdfe"
+          (reference "#PWR033") (unit 1)
+        )
+      )
